Commit message: milestone 3 code

File: body1.urdf (robot description, URDF)
Before this commit: robot robot, 13 links, 12 joints
Links:
- added link BackLeg2, mass 1; collision box size=0.2 1 0.2; visual box size=0.2 1 0.2
- added link FrontLeg2, mass 1; collision box size=0.2 1 0.2; visual box size=0.2 1 0.2
- added link LowerBackLeg2, mass 1; collision box size=0.2 0.2 1; visual box size=0.2 0.2 1
- added link LowerFrontLeg2, mass 1; collision box size=0.2 0.2 1; visual box size=0.2 0.2 1
Joints:
- added joint BackLeg2_LowerBackLeg2: type revolute, parent BackLeg2, child LowerBackLeg2, origin xyz=0 -1 0 rpy=0 0 0, axis 1 0 0, limit lower=-3.14159 upper=3.14159 effort=0.0 velocity=0.0
- added joint FrontLeg2_LowerFrontLeg: type revolute, parent FrontLeg2, child LowerFrontLeg2, origin xyz=0 1 0 rpy=0 0 0, axis 0 0 1, limit lower=-3.14159 upper=3.14159 effort=0.0 velocity=0.0
- added joint Torso_BackLeg2: type revolute, parent Torso, child BackLeg2, origin xyz=0 -0.5 1 rpy=0 0 0, axis 1 0 0, limit lower=-3.14159 upper=3.14159 effort=0.0 velocity=0.0
- added joint Torso_FrontLeg2: type revolute, parent Torso, child FrontLeg2, origin xyz=0 0.5 1 rpy=0 0 0, axis 0 0 1, limit lower=-3.14159 upper=3.14159 effort=0.0 velocity=0.0
- joint BackLeg_LowerBackLeg: axis 3 0 1 -> 1 0 0
- joint FrontLeg_LowerFrontLeg: axis 3 0 1 -> 0 0 1
- joint LeftLeg2_LowerLeftLeg2: axis 3 0 2 -> 1 1 0
- joint LeftLeg_LowerLeftLeg: axis 3 0 2 -> 1 1 0
- joint RightLeg_LowerRightLeg: axis 3 0 2 -> 0 1 1; origin xyz=2 0 0 rpy=0 0 0 -> xyz=1 0 0 rpy=0 0 0
- joint RightLeg_LowerRightLeg2: axis 3 0 2 -> 0 1 1
- joint Torso_BackLeg: axis 3 0 1 -> 1 0 0
- joint Torso_FrontLeg: axis 3 0 1 -> 0 0 1
- joint Torso_LeftLeg: axis 3 0 2 -> 1 1 0
- joint Torso_LeftLeg2: axis 3 0 2 -> 1 1 0
- joint Torso_RightLeg: axis 3 0 2 -> 0 1 1; origin xyz=-0.5 0 1 rpy=0 0 0 -> xyz=0.5 0 1 rpy=0 0 0
- joint Torso_RightLeg2: axis 3 0 2 -> 0 1 1
